File: KiCAD/Instrumentation Amplifier/Instrumentation Amplifier.kicad_sch (KiCad schematic)
At the start: 22 parts, among them U1 OP27, U2 OP27, U3 OP27, U4 OP27, U5 OP27

Commit message: Added title block
Other:
- note added: "26/11/2025"
- note added: "Conor Farrell Breandán Gillanders"
- note added: "Instrumentation Amplifier Circuit"
Changed lines of the file:
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@@
+		)
+	)
+	(text "26/11/2025"
+		(exclude_from_sim no)
+		(at 208.28 193.294 0)
+		(effects
+			(font
+				(size 1.905 1.905)
+				(thickness 0.3175)
+				(color 132 0 0 1)
+			)
+			(justify left)
+		)
+	)
+	(text "Instrumentation Amplifier Circuit"
+		(exclude_from_sim no)
+		(at 188.214 189.738 0)
+		(effects
+			(font
+				(size 2.54 2.54)
+				(thickness 0.3175)
+				(color 132 0 0 1)
+			)
+			(justify left)
+		)
+	)
+	(text "Conor Farrell \nBreandán Gillanders"
+		(exclude_from_sim no)
+		(at 180.594 173.736 0)
+		(effects
+			(font
+				(size 2.54 2.54)
+				(thickness 0.3175)
+				(color 132 0 0 1)
+			)
+			(justify left)
 		)
 	)
